Commit message: Fixed simulation

File: src/velodyne_description/urdf/example.urdf.xacro (robot description, xacro)
@@ -6,10 +6,10 @@
   <link name="base_footprint" />
   <!-- Base Link -->
-  <joint name="footprint" type="fixed" >
+  <!-- <joint name="footprint" type="fixed" >
    <parent link="base_footprint" />
     <child link="base_link" />
     <origin xyz="0 0 0.05" rpy="0 0 0" />
-  </joint>
-  <link name="base_link" >
+  </joint> -->
+  <!-- <link name="base_link" >
     <visual>
       <geometry>
@@ -29,12 +29,12 @@
                izz="3.0" />
     </inertial>
-  </link>
+  </link> -->
   <xacro:include filename="$(find velodyne_description)/urdf/VLP-16.urdf.xacro"/>
-  <xacro:VLP-16 parent="base_link" name="velodyne" topic="/velodyne_points" hz="10" samples="440" gpu="${gpu}">
-    <origin xyz="0 0 0.4" rpy="0 0 0" />
+  <xacro:VLP-16 parent="base_footprint" name="velodyne" topic="/velodyne_points" hz="10" samples="440" gpu="${gpu}">
+    <origin xyz="0 0 0" rpy="0 0 0" />
   </xacro:VLP-16>
-  <xacro:include filename="$(find velodyne_description)/urdf/HDL-32E.urdf.xacro"/>
+  <!-- <xacro:include filename="$(find velodyne_description)/urdf/HDL-32E.urdf.xacro"/>
   <xacro:HDL-32E parent="base_link" name="velodyne2" topic="/velodyne_points2" hz="10" samples="220" gpu="${gpu}">
     <origin xyz="0 0 0.6" rpy="0 0 0" />
-  </xacro:HDL-32E>
+  </xacro:HDL-32E> -->
 </robot>
